Commit message: add missing collision model

File: robots/dyros_assembly_gripper.xacro (robot description, xacro)
@@ -19,4 +19,10 @@
         </material>
       </visual>
+      <collision>
+        <origin xyz="0 0 0" rpy="-1.57 0 -1.57"/>
+        <geometry>
+          <mesh filename="package://assembly_env_description/meshes/gripper_base.stl" scale="0.001 0.001 0.001"/>
+        </geometry>
+      </collision>
       <inertial>
         <mass value="0.55"/>
@@ -27,5 +33,5 @@
       <parent link="${ns}_hand"/>
       <child link="${ns}_finger_right_link"/>
-      <origin xyz="0 -0.000 +0.0745" rpy="0 0 0"/>
+      <origin xyz="0 0.000 +0.0745" rpy="0 0 0"/>
       <axis xyz="0 +1 0"/>
       <limit lower="-0.1" upper="0.15" effort="1000000" velocity="1000000"/>
@@ -41,9 +47,15 @@
         </material>
       </visual>
+      <collision>
+        <origin xyz="0 0 0" rpy="-1.57 0 -1.57"/>
+        <geometry>
+          <mesh filename="package://assembly_env_description/meshes/gripper_tip_right.stl" scale="0.001 0.001 0.001"/>
+        </geometry>
+      </collision>
     </link>
     <joint name="${ns}_finger_left_joint" type="prismatic">
       <parent link="${ns}_hand"/>
       <child link="${ns}_finger_left_link"/>
-      <origin xyz="0 +0.000 +0.0745" rpy="0 0 0"/>
+      <origin xyz="0 0.000 +0.0745" rpy="0 0 0"/>
       <axis xyz="0 -1 0"/>
       <limit lower="-0.1" upper="0.15" effort="1000000" velocity="1000000"/>
@@ -59,4 +71,10 @@
         </material>
       </visual>
+      <collision>
+        <origin xyz="0 0 0" rpy="-1.57 0 -1.57"/>
+        <geometry>
+          <mesh filename="package://assembly_env_description/meshes/gripper_tip_left.stl" scale="0.001 0.001 0.001"/>
+        </geometry>
+      </collision>
     </link>
   </xacro:macro>
