Commit message: update models

File: robots/assembly_env.urdf.xacro (robot description, xacro)
@@ -16,5 +16,5 @@
     </visual>
     <collision>
-      <origin xyz="1.0 0 0.5" rpy="0 0 0"/>
+      <origin xyz="1.0 0 0.5" rpy="0 0 0  "/>
       <geometry>
         <box size="2.4 1.2 1" />
@@ -23,8 +23,11 @@
   </link>
   <!-- left arm with gripper -->
+  <!-- 007853982 -->
   <xacro:panda_arm arm_id="panda_left" connected_to="base"  xyz="0 0.3 1" />
-  <xacro:dyros_assembly_gripper ns="panda_left" rpy="0 0 ${-pi/4}" connected_to="panda_left_link8" />
+  <!-- <xacro:dyros_assembly_gripper ns="panda_left" rpy="0 0 ${-pi/4}" connected_to="panda_left_link8" /> -->
+  <xacro:hand ns="panda_left" rpy="0 0 ${-pi/4}" connected_to="panda_left_link8" />
   <!-- right arm with gripper -->
   <xacro:panda_arm arm_id="panda_right" connected_to="base"  xyz="0 -0.3 1" />
   <xacro:dyros_assembly_gripper ns="panda_right" rpy="0 0 ${-pi/4}" connected_to="panda_right_link8" />
+  <!-- <xacro:hand ns="panda_right" rpy="0 0 ${-pi/4}" connected_to="panda_right_link8" /> -->
 </robot>

File: robots/dyros_assembly_gripper.xacro (robot description, xacro)
@@ -21,19 +21,37 @@
       <inertial>
         <mass value="0.55"/>
-        <inertia ixx="0.0014362" ixy="0.000013" ixz="-0.0000278" iyy="0.00077" iyz="-0.0000897" izz="0.001039"/>
+        <inertia ixx="0.0014362" ixy="0.000013" ixz="-0.0000278" iyy="0.00077" iyz="-0.0000000" izz="0.001039"/>
       </inertial>
     </link>
-    <joint name="${ns}_finger_joint" type="prismatic">
+    <joint name="${ns}_finger_right_joint" type="prismatic">
       <parent link="${ns}_hand"/>
-      <child link="${ns}_finger"/>
-      <origin xyz="-0.01175 -0.0165 +0.0685" rpy="0 0 0"/>
-      <axis xyz="0 1 0"/>
-      <limit lower="0.0" upper="0.15" effort="1000000" velocity="1000000"/>
+      <child link="${ns}_finger_right_link"/>
+      <origin xyz="0 -0.000 +0.0745" rpy="0 0 0"/>
+      <axis xyz="0 +1 0"/>
+      <limit lower="-0.1" upper="0.15" effort="1000000" velocity="1000000"/>
     </joint>
-    <link name="${ns}_finger">
+    <link name="${ns}_finger_right_link">
       <visual>
         <origin xyz="0 0 0" rpy="-1.57 0 -1.57"/>
         <geometry>
-          <mesh filename="package://assembly_env_description/meshes/gripper_moving_tip.stl" scale="0.001 0.001 0.001"/>
+          <mesh filename="package://assembly_env_description/meshes/gripper_tip_right.stl" scale="0.001 0.001 0.001"/>
+        </geometry>
+        <material name="green">
+          <color rgba="0 0.8 0 1"/>
+        </material>
+      </visual>
+    </link>
+    <joint name="${ns}_finger_left_joint" type="prismatic">
+      <parent link="${ns}_hand"/>
+      <child link="${ns}_finger_left_link"/>
+      <origin xyz="0 +0.000 +0.0745" rpy="0 0 0"/>
+      <axis xyz="0 -1 0"/>
+      <limit lower="-0.1" upper="0.15" effort="1000000" velocity="1000000"/>
+    </joint>
+    <link name="${ns}_finger_left_link">
+      <visual>
+        <origin xyz="0 0 0" rpy="-1.57 0 -1.57"/>
+        <geometry>
+          <mesh filename="package://assembly_env_description/meshes/gripper_tip_left.stl" scale="0.001 0.001 0.001"/>
         </geometry>
         <material name="green">

Commit message: add thrid arm

File: robots/assembly_env.urdf.xacro (robot description, xacro)
@@ -4,10 +4,10 @@
   <xacro:include filename="$(find franka_description)/robots/hand.xacro"/>
   <xacro:include filename="dyros_assembly_gripper.xacro"/>
-  <!-- box shaped table as base for the 2 Pandas -->
+  <!-- box shaped table as base for the 3 Pandas -->
   <link name="base">
     <visual>
-      <origin xyz="1.0 0 0.5" rpy="0 0 0"/>
+      <origin xyz="0.4 0 0.5" rpy="0 0 0"/>
       <geometry>
-        <box size="2.4 1.2 1" />
+        <box size="2.7 1.2 1" />
       </geometry>
       <material name="White">
@@ -16,7 +16,7 @@
     </visual>
     <collision>
-      <origin xyz="1.0 0 0.5" rpy="0 0 0  "/>
+      <origin xyz="0.4 0 0.5" rpy="0 0 0  "/>
       <geometry>
-        <box size="2.4 1.2 1" />
+        <box size="2.7 1.2 1" />
       </geometry>
     </collision>
@@ -31,3 +31,6 @@
   <xacro:dyros_assembly_gripper ns="panda_right" rpy="0 0 ${-pi/4}" connected_to="panda_right_link8" />
   <!-- <xacro:hand ns="panda_right" rpy="0 0 ${-pi/4}" connected_to="panda_right_link8" /> -->
+   <!-- top arm with gripper -->
+  <xacro:panda_arm arm_id="panda_top" connected_to="base"  xyz="1.525 0 1" rpy="0 0 ${pi}" />
+  <xacro:hand ns="panda_top" rpy="0 0 ${-pi/4}" connected_to="panda_top_link8" />
 </robot>
