Commit message: update gripper col model

File: robots/dyros_assembly_gripper2.xacro (robot description, xacro)
@@ -20,7 +20,7 @@
       </visual>
       <collision>
-        <origin xyz="0 0 0" rpy="-1.57 0 -1.57"/>
+        <origin xyz="0.017 0 0.029" rpy="0 0 0"/>
         <geometry>
-          <mesh filename="package://assembly_env_description/meshes/gripper2_base.stl" scale="0.001 0.001 0.001"/>
+          <box size="0.125 0.21 0.06"/>
         </geometry>
       </collision>
@@ -48,7 +48,7 @@
       </visual>
       <collision>
-        <origin xyz="0 0 0" rpy="-1.57 0 -1.57"/>
+        <origin xyz="0 0 0.01" rpy="0 0 0"/>
         <geometry>
-          <mesh filename="package://assembly_env_description/meshes/gripper2_tip.stl" scale="0.001 0.001 0.001"/>
+          <box size="0.08 0.0185 0.035"/>
         </geometry>
       </collision>
@@ -72,7 +72,7 @@
       </visual>
       <collision>
-        <origin xyz="0 0 0" rpy="-1.57 0 -1.57"/>
+        <origin xyz="0 0 0.01" rpy="0 0 0"/>
         <geometry>
-          <mesh filename="package://assembly_env_description/meshes/gripper2_tip.stl" scale="0.001 0.001 0.001"/>
+          <box size="0.08 0.0185 0.035"/>
         </geometry>
       </collision>

Commit message: add tcp

File: robots/dyros_assembly_gripper2.xacro (robot description, xacro)
@@ -1,5 +1,5 @@
 <?xml version="1.0"?>
 <robot xmlns:xacro="http://www.ros.org/wiki/xacro" name="dyros_assembly_gripper2">
-  <xacro:macro name="dyros_assembly_gripper2" params="connected_to:='' ns:='' rpy:='0 0 0' xyz:='0 0 0' ">
+  <xacro:macro name="dyros_assembly_gripper2" params="connected_to:='' ns:='' rpy:='0 0 0' xyz:='0 0 0' tcp_xyz:='0 0 0.0825' tcp_rpy:='0 0 0' ">
     <xacro:unless value="${connected_to == ''}">
       <joint name="${ns}_hand_joint" type="fixed">
@@ -30,4 +30,11 @@
       </inertial>
     </link>
+    <!-- Define the hand_tcp frame -->
+    <link name="${ns}_hand_tcp" />
+    <joint name="${ns}_hand_tcp_joint" type="fixed">
+      <origin xyz="${tcp_xyz}" rpy="${tcp_rpy}" />
+      <parent link="${ns}_hand" />
+      <child link="${ns}_hand_tcp" />
+    </joint>
     <joint name="${ns}_finger_right_joint" type="prismatic">
       <parent link="${ns}_hand"/>
